File: Instrumentation Control R1.kicad_sch (KiCad schematic)
At the start: 100 parts, among them J11 Conn_01x04_Pin, J12 Conn_01x04_Pin, J13 Conn_01x05_Pin, J14 Conn_01x05_Pin, J15 Conn_01x06_Pin, J17 Conn_01x03_Pin, J19 Conn_02x04_Top_Bottom, Q2 NMOS, Q3 NMOS, Q4 NMOS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

Commit message: Added USB-UART Bridge
Parts:
- removed C101: 0.1uF, Capacitor_SMD:C_0805_2012Metric, symbol Device:C
- removed C102: 1uF, Capacitor_SMD:C_0805_2012Metric, symbol Device:C
- removed J13: Conn_01x05_Pin, Connector_JST:JST_PH_B5B-PH-K_1x05_P2.00mm_Vertical, symbol Connector_Generic:Conn_01x05
Other:
- note added: "Headers & Mounting Holes"
- note removed: "Headers"
- moved on the sheet: C103, C104, H1, H2, H3, H4, J14

Commit message: Final updates for R2
Other:
- sheet MCU ports: added none; removed USART1_CK, USART1_RX, USART1_TX
Changed lines of the file:
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@@
 	(wire
 		(pts
-			(xy 33.02 45.72) (xy 39.37 45.72)
-		)
-		(stroke
-			(width 0)
-			(type default)
-		)
-	)
-	(wire
-		(pts
 			(xy 86.36 66.04) (xy 115.57 66.04)
 		)
@@
 	(wire
 		(pts
-			(xy 33.02 54.61) (xy 39.37 54.61)
+			(xy 34.29 45.72) (xy 39.37 45.72)
 		)
 		(stroke
@@
 	(wire
 		(pts
-			(xy 33.02 63.5) (xy 39.37 63.5)
+			(xy 34.29 54.61) (xy 39.37 54.61)
 		)
 		(stroke
@@
 	(wire
 		(pts
-			(xy 33.02 43.18) (xy 39.37 43.18)
-		)
-		(stroke
-			(width 0)
-			(type default)
-		)
-	)
-	(wire
-		(pts
 			(xy 342.9 87.63) (xy 342.9 107.95)
 		)
@@
 	(wire
 		(pts
-			(xy 33.02 52.07) (xy 39.37 52.07)
+			(xy 34.29 43.18) (xy 39.37 43.18)
 		)
 		(stroke
@@
 	(wire
 		(pts
-			(xy 33.02 48.26) (xy 39.37 48.26)
-		)
-		(stroke
-			(width 0)
-			(type default)
-		)
-	)
-	(wire
-		(pts
 			(xy 247.65 213.36) (xy 250.19 213.36)
 		)
@@
 	(wire
 		(pts
-			(xy 33.02 66.04) (xy 39.37 66.04)
+			(xy 34.29 57.15) (xy 39.37 57.15)
 		)
 		(stroke
@@
 	(wire
 		(pts
-			(xy 33.02 60.96) (xy 39.37 60.96)
+			(xy 34.29 52.07) (xy 39.37 52.07)
 		)
 		(stroke
@@
 	(wire
 		(pts
-			(xy 33.02 57.15) (xy 39.37 57.15)
+			(xy 34.29 48.26) (xy 39.37 48.26)
 		)
 		(stroke
@@
 	)
 	(label "RST"
-		(at 33.02 66.04 180)
+		(at 34.29 57.15 180)
 		(effects
 			(font
@@
 	)
 	(label "PA0{slash}WKUP"
-		(at 33.02 60.96 180)
+		(at 34.29 52.07 180)
 		(effects
 			(font
@@
 	)
 	(label "SYNC"
-		(at 33.02 63.5 180)
+		(at 34.29 54.61 180)
 		(effects
 			(font
@@
 		)
 	)
-	(label "USART1_CK"
-		(at 33.02 48.26 180)
-		(effects
-			(font
-				(size 1.27 1.27)
-			)
-			(justify right bottom)
-		)
-	)
 	(label "SYNC"
 		(at 198.12 162.56 180)
@@
 	)
 	(label "USART2_RX"
-		(at 33.02 54.61 180)
+		(at 34.29 45.72 180)
 		(effects
 			(font
@@
 	)
 	(label "USART2_CK"
-		(at 33.02 57.15 180)
+		(at 34.29 48.26 180)
 		(effects
 			(font
@@
 	)
 	(label "USART2_TX"
-		(at 33.02 52.07 180)
+		(at 34.29 43.18 180)
 		(effects
 			(font
@@
 		)
 	)
-	(label "USART1_TX"
-		(at 33.02 43.18 180)
-		(effects
-			(font
-				(size 1.27 1.27)
-			)
-			(justify right bottom)
-		)
-	)
 	(label "SLOT7_CS"
 		(at 138.43 66.04 0)
@@
 		)
 	)
-	(label "USART1_RX"
-		(at 33.02 45.72 180)
-		(effects
-			(font
-				(size 1.27 1.27)
-			)
-			(justify right bottom)
-		)
-	)
 	(label "CAN_H"
 		(at 379.73 55.88 0)
@@
 		)
 		(pin "PA15" bidirectional
-			(at 39.37 66.04 180)
+			(at 39.37 57.15 180)
 			(effects
 				(font
@@
 		)
 		(pin "USART2_RX" input
-			(at 39.37 54.61 180)
+			(at 39.37 45.72 180)
 			(effects
 				(font
@@
 		)
 		(pin "USART2_CK" output
-			(at 39.37 57.15 180)
+			(at 39.37 48.26 180)
 			(effects
 				(font
@@
 		)
 		(pin "PA1" bidirectional
-			(at 39.37 63.5 180)
+			(at 39.37 54.61 180)
 			(effects
 				(font
@@
 		)
 		(pin "PA0" bidirectional
-			(at 39.37 60.96 180)
+			(at 39.37 52.07 180)
 			(effects
 				(font
@@
 		)
 		(pin "USART2_TX" output
-			(at 39.37 52.07 180)
+			(at 39.37 43.18 180)
 			(effects
 				(font
@@
 			)
 		)
-		(pin "USART1_CK" output
-			(at 39.37 48.26 180)
-			(effects
-				(font
-					(size 1.27 1.27)
-				)
-				(justify left)
-			)
-		)
 		(pin "MISO_1" input
 			(at 86.36 50.8 0)
@@
 			)
 		)
-		(pin "USART1_RX" input
-			(at 39.37 45.72 180)
-			(effects
-				(font
-					(size 1.27 1.27)
-				)
-				(justify left)
-			)
-		)
-		(pin "USART1_TX" output
-			(at 39.37 43.18 180)
-			(effects
-				(font
-					(size 1.27 1.27)
-				)
-				(justify left)
-			)
-		)

Commit message: libraries
Parts:
- D41, D42, D43, D44, D45, D46, D47, D48: value LED -> LED_R
Changed lines of the file:
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@@
 			)
 		)
-		(property "Value" "LED"
+		(property "Value" "LED_R"
 			(at 153.67 199.7074 90)
 			(effects
@@
 			)
 		)
-		(property "Value" "LED"
+		(property "Value" "LED_R"
 			(at 350.52 199.7074 90)
 			(effects
@@
 			)
 		)
-		(property "Value" "LED"
+		(property "Value" "LED_R"
 			(at 114.3 199.7074 90)
 			(effects
@@
 			)
 		)
-		(property "Value" "LED"
+		(property "Value" "LED_R"
 			(at 271.78 199.7074 90)
 			(effects
@@
 			)
 		)
-		(property "Value" "LED"
+		(property "Value" "LED_R"
 			(at 311.15 199.7074 90)
 			(effects
@@
 			)
 		)
-		(property "Value" "LED"
+		(property "Value" "LED_R"
 			(at 389.89 199.7074 90)
 			(effects
@@
 			)
 		)
-		(property "Value" "LED"
+		(property "Value" "LED_R"
 			(at 232.41 199.7074 90)
 			(effects
@@
 			)
 		)
-		(property "Value" "LED"
+		(property "Value" "LED_R"
 			(at 193.04 199.7074 90)
 			(effects
