File: MCU.kicad_sch (KiCad schematic)
At the start: 81 parts, among them J13 2068320402, J3 FTSH-107-01-L-D-K, J4 USB_C_Receptacle_USB2.0_16P, Q1 PMOS, Q10 NMOS, SW2 SW_Push, U1 MCP2562-E-SN, U13 TPD2EUSB30, U14 MAX40200AUK, U15 MAX40200AUK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

Commit message: Library updates
Parts:
- J3: symbol Connector:FTSH-107-01-L-D-K -> Symbols:FTSH-107-01-L-D-K
Changed lines of the file:
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@@
 	)
 	(symbol
-		(lib_id "Connector:FTSH-107-01-L-D-K")
-		(at 167.64 177.8 0)
+		(lib_id "Symbols:FTSH-107-01-L-D-K")
+		(at 165.1 177.8 0)
 		(unit 1)
 		(exclude_from_sim no)
@@
 		)
 		(property "Footprint" "Footprints:SAMTEC_FTSH-107-01-L-D-K"
-			(at 167.64 177.8 0)
+			(at 165.1 177.8 0)
 			(effects
 				(font
@@
 		)
 		(property "Datasheet" ""
-			(at 167.64 177.8 0)
+			(at 165.1 177.8 0)
 			(effects
 				(font
@@
 		)
 		(property "Description" ""
-			(at 167.64 177.8 0)
+			(at 165.1 177.8 0)
 			(effects
 				(font
@@
 		)
 		(property "MAXIMUM_PACKAGE_HEIGHT" "5.71mm"
-			(at 167.64 177.8 0)
+			(at 165.1 177.8 0)
 			(effects
 				(font
@@
 		)
 		(property "CREATOR" "AMINA"
-			(at 167.64 177.8 0)
+			(at 165.1 177.8 0)
 			(effects
 				(font
@@
 		)
 		(property "STANDARD" "Manufacturer Recommendations"
-			(at 167.64 177.8 0)
+			(at 165.1 177.8 0)
 			(effects
 				(font
@@
 		)
 		(property "PARTREV" "B"
-			(at 167.64 177.8 0)
+			(at 165.1 177.8 0)
 			(effects
 				(font
@@
 		)
 		(property "VERIFIER" "Your name, use the same always"
-			(at 167.64 177.8 0)
+			(at 165.1 177.8 0)
 			(effects
 				(font
@@
 		)
 		(property "MANUFACTURER" "Samtec"
-			(at 167.64 177.8 0)
+			(at 165.1 177.8 0)
 			(effects
 				(font
