File: MCU.kicad_sch (KiCad schematic)
At the start: 34 parts, among them J3 FTSH-107-01-L-D-K, SW2 SW_Push, U1 MCP2562-E-SN, U4 STM32F103C8Tx, Y3 8MHz, Y4 32.768K

Commit message: Updated
Parts:
- added R7: 33K, Resistor_SMD:R_0805_2012Metric, symbol Device:R
- added R8: 20K, Resistor_SMD:R_0805_2012Metric, symbol Device:R
Connections:
- net +5V: now also R7.1
- net GND: now also R8.2
- net PA0 renamed VSENS
- net VSENS: now also R7.2, R8.1
Other:
- moved on the sheet: R14

Commit message: Final updates for R2
Parts:
- added C3: 47nF, Capacitor_SMD:C_0805_2012Metric, symbol Device:C
Connections:
- net GND: now also C3.2
- net VSENS: now also C3.1
Changed lines of the file:
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@@
 	(wire
 		(pts
+			(xy 50.8 107.95) (xy 43.18 107.95)
+		)
+		(stroke
+			(width 0)
+			(type default)
+		)
+	)
+	(wire
+		(pts
 			(xy 163.83 85.09) (xy 163.83 86.36)
 		)
@@
 	(wire
 		(pts
+			(xy 43.18 107.95) (xy 43.18 109.22)
+		)
+		(stroke
+			(width 0)
+			(type default)
+		)
+	)
+	(wire
+		(pts
 			(xy 41.91 77.47) (xy 57.15 77.47)
 		)
@@
 	(wire
 		(pts
+			(xy 43.18 116.84) (xy 43.18 118.11)
+		)
+		(stroke
+			(width 0)
+			(type default)
+		)
+	)
+	(wire
+		(pts
 			(xy 74.93 33.02) (xy 74.93 34.29)
 		)
@@
 	)
 	(symbol
+		(lib_id "power:GND")
+		(at 43.18 118.11 0)
+		(unit 1)
+		(exclude_from_sim no)
+		(in_bom yes)
+		(on_board yes)
+		(dnp no)
+		(fields_autoplaced yes)
+		(property "Reference" "#PWR097"
+			(at 43.18 124.46 0)
+			(effects
+				(font
+					(size 1.27 1.27)
+				)
+				(hide yes)
+			)
+		)
+		(property "Value" "GND"
+			(at 43.18 123.19 0)
+			(effects
+				(font
+					(size 1.27 1.27)
+				)
+			)
+		)
+		(property "Footprint" ""
+			(at 43.18 118.11 0)
+			(effects
+				(font
+					(size 1.27 1.27)
+				)
+				(hide yes)
+			)
+		)
+		(property "Datasheet" ""
+			(at 43.18 118.11 0)
+			(effects
+				(font
+					(size 1.27 1.27)
+				)
+				(hide yes)
+			)
+		)
+		(property "Description" "Power symbol creates a global label with name \"GND\" , ground"
+			(at 43.18 118.11 0)
+			(effects
+				(font
+					(size 1.27 1.27)
+				)
+				(hide yes)
+			)
+		)
+		(pin "1"
+		)
+		(instances
+			(project "Pump Control Card R1"
+				(path "/ff1870f3-6a64-4f6c-9ec6-b3e6f5db28b5/1f0089c3-1425-4c68-94bd-e8236ea2ca92"
+					(reference "#PWR097")
+					(unit 1)
+				)
+			)
+		)
+	)
+	(symbol
 		(lib_id "power:+3.3V")
 		(at 41.91 67.31 0)
@@
 					(unit 1)
 				)
+			)
+		)
+	)
+	(symbol
+		(lib_id "Device:C")
+		(at 43.18 113.03 0)
+		(unit 1)
+		(exclude_from_sim no)
+		(in_bom yes)
+		(on_board yes)
+		(dnp no)
+		(property "Reference" "C3"
+			(at 43.434 110.998 0)
+			(effects
+				(font
+					(size 1.27 1.27)
+				)
+				(justify left)
+			)
+		)
+		(property "Value" "47nF"
+			(at 43.434 115.316 0)
+			(effects
+				(font
+					(size 1.27 1.27)
+				)
+				(justify left)
+			)
+		)
+		(property "Footprint" "Capacitor_SMD:C_0805_2012Metric"
+			(at 44.1452 116.84 0)
+			(effects
+				(font
+					(size 1.27 1.27)
+				)
+				(hide yes)
+			)
+		)
+		(property "Datasheet" "~"
+			(at 43.18 113.03 0)
+			(effects
+				(font
+					(size 1.27 1.27)
+				)
+				(hide yes)
+			)
+		)
+		(property "Description" "Unpolarized capacitor"
+			(at 43.18 113.03 0)
+			(effects
+				(font
+					(size 1.27 1.27)
+				)
+				(hide yes)
+			)
+		)
+		(pin "2"
+		)
+		(pin "1"
+		)
+		(instances
+			(project "Pump Control Card R1"
+				(path "/ff1870f3-6a64-4f6c-9ec6-b3e6f5db28b5/1f0089c3-1425-4c68-94bd-e8236ea2ca92"
+					(reference "C3")
+					(unit 1)
+				)

Commit message: Library updates
Parts:
- J3: footprint Connector_Samtec:SAMTEC_FTSH-107-01-L-D-K -> Footprints:SAMTEC_FTSH-107-01-L-D-K; symbol Connector:FTSH-107-01-L-D-K -> Symbols:FTSH-107-01-L-D-K
Changed lines of the file:
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@@
 	(wire
 		(pts
+			(xy 173.99 44.45) (xy 177.8 44.45)
+		)
+		(stroke
+			(width 0)
+			(type default)
+		)
+	)
+	(wire
+		(pts
 			(xy 111.76 80.01) (xy 115.57 80.01)
 		)
@@
 	(wire
 		(pts
-			(xy 173.99 44.45) (xy 177.8 44.45)
-		)
-		(stroke
-			(width 0)
-			(type default)
-		)
-	)
-	(wire
-		(pts
 			(xy 153.67 76.2) (xy 153.67 77.47)
 		)
@@
 	)
 	(symbol
-		(lib_id "Connector:FTSH-107-01-L-D-K")
-		(at 167.64 39.37 0)
+		(lib_id "Symbols:FTSH-107-01-L-D-K")
+		(at 165.1 39.37 0)
 		(unit 1)
 		(exclude_from_sim no)
@@
 			)
 		)
-		(property "Footprint" "Connector_Samtec:SAMTEC_FTSH-107-01-L-D-K"
-			(at 167.64 39.37 0)
+		(property "Footprint" "Footprints:SAMTEC_FTSH-107-01-L-D-K"
+			(at 165.1 39.37 0)
 			(effects
 				(font
@@
 		)
 		(property "Datasheet" ""
-			(at 167.64 39.37 0)
+			(at 165.1 39.37 0)
 			(effects
 				(font
@@
 		)
 		(property "Description" ""
-			(at 167.64 39.37 0)
+			(at 165.1 39.37 0)
 			(effects
 				(font
@@
 		)
 		(property "MAXIMUM_PACKAGE_HEIGHT" "5.71mm"
-			(at 167.64 39.37 0)
+			(at 165.1 39.37 0)
 			(effects
 				(font
@@
 		)
 		(property "CREATOR" "AMINA"
-			(at 167.64 39.37 0)
+			(at 165.1 39.37 0)
 			(effects
 				(font
@@
 		)
 		(property "STANDARD" "Manufacturer Recommendations"
-			(at 167.64 39.37 0)
+			(at 165.1 39.37 0)
 			(effects
 				(font
@@
 		)
 		(property "PARTREV" "B"
-			(at 167.64 39.37 0)
+			(at 165.1 39.37 0)
 			(effects
 				(font
@@
 		)
 		(property "VERIFIER" "Your name, use the same always"
-			(at 167.64 39.37 0)
+			(at 165.1 39.37 0)
 			(effects
 				(font
@@
 		)
 		(property "MANUFACTURER" "Samtec"
-			(at 167.64 39.37 0)
+			(at 165.1 39.37 0)
 			(effects
 				(font
