File: PCIe.kicad_sch (KiCad schematic)
At the start: 15 parts, among them J10 10018784-10201TLF

Commit message: Final updates for R2
Changed lines of the file:
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@@
 	)
 	(hierarchical_label "IRQ_OUT"
-		(shape input)
+		(shape output)
 		(at 111.76 133.35 180)
 		(effects

Commit message: libraries
Parts:
- D13: value LED -> LED_B
- D38: value D_Zener -> D_3V3
- D39: value D_Zener -> D_VIN
- D40: value D_Zener -> D_5V
Changed lines of the file:
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@@
 			)
 		)
-		(property "Value" "LED"
+		(property "Value" "LED_B"
 			(at 95.25 86.6774 90)
 			(effects
@@
 			)
 		)
-		(property "Value" "D_Zener"
-			(at 101.346 102.616 90)
+		(property "Value" "D_VIN"
+			(at 102.87 103.124 90)
 			(effects
 				(font
@@
 			)
 		)
-		(property "Value" "D_Zener"
-			(at 101.092 59.436 90)
+		(property "Value" "D_3V3"
+			(at 102.87 59.944 90)
 			(effects
 				(font
@@
 			)
 		)
-		(property "Value" "D_Zener"
-			(at 97.282 79.756 90)
-			(effects
-				(font
+		(property "Value" "D_5V"
+			(at 100.33 80.264 90)
+			(effects
+				(font

Commit message: library updates
Parts:
- J10: footprint Connector_PCBEdge:CONN_10018784-10201TLF -> Footprints:CONN_10018784-10201TLF; symbol Connector:10018784-10201TLF -> Symbols:10018784-10201TLF
Changed lines of the file:
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@@
 	)
 	(symbol
-		(lib_id "Connector:10018784-10201TLF")
+		(lib_id "Symbols:10018784-10201TLF")
 		(at 128.27 92.71 0)
 		(unit 1)
@@
 			)
 		)
-		(property "Footprint" "Connector_PCBEdge:CONN_10018784-10201TLF"
+		(property "Footprint" "Footprints:CONN_10018784-10201TLF"
 			(at 128.27 92.71 0)
 			(effects

Commit message: Updated libraries
Parts:
- J10: symbol Symbols:10018784-10201TLF -> Connector:10018784-10201TLF
Changed lines of the file:
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@@
 	)
 	(symbol
-		(lib_id "Symbols:10018784-10201TLF")
+		(lib_id "Connector:10018784-10201TLF")
 		(at 128.27 92.71 0)
 		(unit 1)

Commit message: Library updates
Parts:
- J10: symbol Connector:10018784-10201TLF -> Symbols:10018784-10201TLF
Changed lines of the file:
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@@
 	)
 	(symbol
-		(lib_id "Connector:10018784-10201TLF")
+		(lib_id "Symbols:10018784-10201TLF")
 		(at 128.27 92.71 0)
 		(unit 1)
