File: PCIe.kicad_sch (KiCad schematic)
At the start: 7 parts, among them J10 10018784-10201TLF

Commit message: Updated libraries
Parts:
- J10: symbol Connector:10018784-10201TLF -> Symbols:10018784-10201TLF
Changed lines of the file:
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@@
 	)
 	(symbol
-		(lib_id "Connector:10018784-10201TLF")
+		(lib_id "Symbols:10018784-10201TLF")
 		(at 128.27 92.71 0)
 		(unit 1)
