File: PCIe2.kicad_sch (KiCad schematic)
At the start: 18 parts, among them J1 10018784-10201TLF, U3 74LVC1G32

Commit message: libraries
Parts:
- D1: value LED -> LED_B
- D17: value D_Zener -> D_3V3
- D18: value D_Zener -> D_VIN
- D19: value D_Zener -> D_5V
Changed lines of the file:
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@@
 			)
 		)
-		(property "Value" "D_Zener"
+		(property "Value" "D_3V3"
 			(at 106.68 58.4199 90)
 			(effects
@@
 			)
 		)
-		(property "Value" "D_Zener"
+		(property "Value" "D_5V"
 			(at 102.87 78.7399 90)
 			(effects
@@
 			)
 		)
-		(property "Value" "LED"
+		(property "Value" "LED_B"
 			(at 95.25 86.6774 90)
 			(effects
@@
 			)
 		)
-		(property "Value" "D_Zener"
+		(property "Value" "D_VIN"
 			(at 106.68 101.5999 90)
 			(effects

Commit message: library updates
Parts:
- J1: footprint Connector_PCBEdge:CONN_10018784-10201TLF -> Footprints:CONN_10018784-10201TLF; symbol Connector:10018784-10201TLF -> Symbols:10018784-10201TLF
Changed lines of the file:
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@@
 	)
 	(symbol
-		(lib_id "Connector:10018784-10201TLF")
+		(lib_id "Symbols:10018784-10201TLF")
 		(at 128.27 92.71 0)
 		(unit 1)
@@
 			)
 		)
-		(property "Footprint" "Connector_PCBEdge:CONN_10018784-10201TLF"
+		(property "Footprint" "Footprints:CONN_10018784-10201TLF"
 			(at 128.27 92.71 0)
 			(effects

Commit message: Updated libraries
Parts:
- J1: symbol Symbols:10018784-10201TLF -> Connector:10018784-10201TLF
Changed lines of the file:
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@@
 	)
 	(symbol
-		(lib_id "Symbols:10018784-10201TLF")
+		(lib_id "Connector:10018784-10201TLF")
 		(at 128.27 92.71 0)
 		(unit 1)

Commit message: Library updates
Parts:
- J1: symbol Connector:10018784-10201TLF -> Symbols:10018784-10201TLF
Changed lines of the file:
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@@
 	)
 	(symbol
-		(lib_id "Connector:10018784-10201TLF")
+		(lib_id "Symbols:10018784-10201TLF")
 		(at 128.27 92.71 0)
 		(unit 1)
