File: Buffer_3V3.kicad_sch (KiCad schematic)
At the start: 16 parts, among them U10 74AHC125, U7 74AHC125, U8 74AHC125, U9 74AHC125

Commit message: Updated libraries
Parts:
- R20, R21, R22, R23: footprint Resistor_SMD:EXB28V_PAN -> Footprints:EXB28V_PAN; symbol Device:EXB-28V220JX -> Symbols:EXB-28V220JX
Changed lines of the file:
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@@
 	)
 	(symbol
-		(lib_id "Device:EXB-28V220JX")
+		(lib_id "Symbols:EXB-28V220JX")
 		(at 177.8 109.22 0)
 		(unit 1)
@@
 			)
 		)
-		(property "Footprint" "Resistor_SMD:EXB28V_PAN"
+		(property "Footprint" "Footprints:EXB28V_PAN"
 			(at 177.8 109.22 0)
 			(effects
@@
 	)
 	(symbol
-		(lib_id "Device:EXB-28V220JX")
+		(lib_id "Symbols:EXB-28V220JX")
 		(at 236.22 109.22 0)
 		(unit 1)
@@
 			)
 		)
-		(property "Footprint" "Resistor_SMD:EXB28V_PAN"
+		(property "Footprint" "Footprints:EXB28V_PAN"
 			(at 236.22 109.22 0)
 			(effects
@@
 	)
 	(symbol
-		(lib_id "Device:EXB-28V220JX")
+		(lib_id "Symbols:EXB-28V220JX")
 		(at 59.69 109.22 0)
 		(unit 1)
@@
 			)
 		)
-		(property "Footprint" "Resistor_SMD:EXB28V_PAN"
+		(property "Footprint" "Footprints:EXB28V_PAN"
 			(at 59.69 109.22 0)
 			(effects
@@
 	)
 	(symbol
-		(lib_id "Device:EXB-28V220JX")
+		(lib_id "Symbols:EXB-28V220JX")
 		(at 118.11 109.22 0)
 		(unit 1)
@@
 			)
 		)
-		(property "Footprint" "Resistor_SMD:EXB28V_PAN"
+		(property "Footprint" "Footprints:EXB28V_PAN"
 			(at 118.11 109.22 0)
 			(effects
