File: Buffer_5V.kicad_sch (KiCad schematic)
At the start: 16 parts, among them U3 74AHCT125, U4 74AHCT125, U5 74AHCT125, U6 74AHCT125

Commit message: Updated libraries
Parts:
- R15, R16, R17, R18: footprint Resistor_SMD:EXB28V_PAN -> Footprints:EXB28V_PAN; symbol Device:EXB-28V220JX -> Symbols:EXB-28V220JX
Changed lines of the file:
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@@
 	)
 	(symbol
-		(lib_id "Device:EXB-28V220JX")
+		(lib_id "Symbols:EXB-28V220JX")
 		(at 113.03 107.95 0)
 		(unit 1)
@@
 			)
 		)
-		(property "Footprint" "Resistor_SMD:EXB28V_PAN"
+		(property "Footprint" "Footprints:EXB28V_PAN"
 			(at 113.03 107.95 0)
 			(effects
@@
 	)
 	(symbol
-		(lib_id "Device:EXB-28V220JX")
+		(lib_id "Symbols:EXB-28V220JX")
 		(at 172.72 107.95 0)
 		(unit 1)
@@
 			)
 		)
-		(property "Footprint" "Resistor_SMD:EXB28V_PAN"
+		(property "Footprint" "Footprints:EXB28V_PAN"
 			(at 172.72 107.95 0)
 			(effects
@@
 	)
 	(symbol
-		(lib_id "Device:EXB-28V220JX")
+		(lib_id "Symbols:EXB-28V220JX")
 		(at 231.14 107.95 0)
 		(unit 1)
@@
 			)
 		)
-		(property "Footprint" "Resistor_SMD:EXB28V_PAN"
+		(property "Footprint" "Footprints:EXB28V_PAN"
 			(at 231.14 107.95 0)
 			(effects
@@
 	)
 	(symbol
-		(lib_id "Device:EXB-28V220JX")
+		(lib_id "Symbols:EXB-28V220JX")
 		(at 54.61 107.95 0)
 		(unit 1)
@@
 			)
 		)
-		(property "Footprint" "Resistor_SMD:EXB28V_PAN"
+		(property "Footprint" "Footprints:EXB28V_PAN"
 			(at 54.61 107.95 0)
 			(effects
