File: Timing Card R1.kicad_sch (KiCad schematic)
At the start: 27 parts, among them J1 71430-0101, J2 Conn_01x10

Commit message: Updated libraries
Parts:
- J1: footprint Connector:MOLEX_71430-0101 -> Footprints:MOLEX_71430-0101; symbol Connector:71430-0101 -> Symbols:71430-0101
Changed lines of the file:
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@@
 	)
 	(no_connect
-		(at 40.64 80.01)
+		(at 40.64 74.93)
 	)
 	(no_connect
-		(at 40.64 74.93)
+		(at 40.64 77.47)
 	)
 	(no_connect
@@
 	)
 	(no_connect
-		(at 40.64 77.47)
+		(at 40.64 62.23)
 	)
 	(no_connect
-		(at 40.64 62.23)
+		(at 40.64 80.01)
 	)
 	(wire
@@
 	(wire
 		(pts
-			(xy 38.1 80.01) (xy 40.64 80.01)
-		)
-		(stroke
-			(width 0)
-			(type default)
-		)
-	)
-	(wire
-		(pts
 			(xy 190.5 134.62) (xy 190.5 142.24)
 		)
@@
 	(wire
 		(pts
+			(xy 38.1 74.93) (xy 40.64 74.93)
+		)
+		(stroke
+			(width 0)
+			(type default)
+		)
+	)
+	(wire
+		(pts
 			(xy 124.46 63.5) (xy 120.65 63.5)
 		)
@@
 	(wire
 		(pts
+			(xy 38.1 80.01) (xy 40.64 80.01)
+		)
+		(stroke
+			(width 0)
+			(type default)
+		)
+	)
+	(wire
+		(pts
 			(xy 218.44 134.62) (xy 233.68 134.62)
 		)
@@
 	(wire
 		(pts
-			(xy 38.1 77.47) (xy 40.64 77.47)
-		)
-		(stroke
-			(width 0)
-			(type default)
-		)
-	)
-	(wire
-		(pts
 			(xy 153.67 171.45) (xy 153.67 172.72)
 		)
@@
 	(wire
 		(pts
+			(xy 38.1 77.47) (xy 40.64 77.47)
+		)
+		(stroke
+			(width 0)
+			(type default)
+		)
+	)
+	(wire
+		(pts
 			(xy 190.5 71.12) (xy 193.04 71.12)
 		)
@@
 	(wire
 		(pts
-			(xy 38.1 74.93) (xy 40.64 74.93)
-		)
-		(stroke
-			(width 0)
-			(type default)
-		)
-	)
-	(wire
-		(pts
 			(xy 55.88 35.56) (xy 67.31 35.56)
 		)
@@
 	)
 	(symbol
-		(lib_id "Connector:71430-0101")
+		(lib_id "Symbols:71430-0101")
 		(at 205.74 106.68 0)
 		(unit 1)
@@
 			)
 		)
-		(property "Footprint" "Connector:MOLEX_71430-0101"
+		(property "Footprint" "Footprints:MOLEX_71430-0101"
 			(at 205.74 106.68 0)
 			(effects
