File: Camera-Control-Card/PCIe.kicad_sch (KiCad schematic)
At the start: 7 parts, among them J10 10018784-10201TLF

Commit message: test
Parts:
- removed C91: 0.1uF, Capacitor_SMD:C_0805_2012Metric, symbol Device:C
- removed C93: 1uF, Capacitor_SMD:C_0805_2012Metric, symbol Device:C
- removed C96: 10uF, Capacitor_SMD:CP_Elec_6.3x5.9, symbol Device:C
- C88, C89: footprint Capacitor_SMD:C_0805_2012Metric -> Capacitor_SMD:C_0603_1608Metric
Connections:
- removed net +5V: J10.A10, J10.A11, J10.A12, J10.A13, J10.A14, J10.A15, J10.A9
- no-connect marks 8 -> 15

Commit message: Updates
Parts:
- renumbered C88 to C1, C89 to C2, C90 to C3, J10 to J8
Other:
- moved on the sheet: C1, C2, C3
Changed lines of the file:
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@@
 	)
 	(junction
-		(at 161.29 43.18)
+		(at 168.91 52.07)
 		(diameter 0)
 		(color 0 0 0 0)
@@
 	)
 	(junction
-		(at 161.29 53.34)
+		(at 168.91 62.23)
 		(diameter 0)
 		(color 0 0 0 0)
@@
 	(junction
 		(at 102.87 123.19)
+		(diameter 0)
+		(color 0 0 0 0)
+	)
+	(junction
+		(at 157.48 52.07)
 		(diameter 0)
 		(color 0 0 0 0)
@@
 	(wire
 		(pts
-			(xy 172.72 52.07) (xy 172.72 53.34)
+			(xy 180.34 60.96) (xy 180.34 62.23)
 		)
 		(stroke
@@
 	(wire
 		(pts
-			(xy 161.29 43.18) (xy 172.72 43.18)
+			(xy 168.91 52.07) (xy 180.34 52.07)
 		)
 		(stroke
@@
 	(wire
 		(pts
-			(xy 161.29 43.18) (xy 161.29 44.45)
+			(xy 168.91 52.07) (xy 168.91 53.34)
 		)
 		(stroke
@@
 	(wire
 		(pts
-			(xy 172.72 43.18) (xy 172.72 44.45)
+			(xy 180.34 52.07) (xy 180.34 53.34)
 		)
 		(stroke
@@
 	(wire
 		(pts
+			(xy 143.51 52.07) (xy 157.48 52.07)
+		)
+		(stroke
+			(width 0)
+			(type default)
+		)
+	)
+	(wire
+		(pts
 			(xy 113.03 85.09) (xy 115.57 85.09)
 		)
@@
 	(wire
 		(pts
-			(xy 149.86 43.18) (xy 161.29 43.18)
+			(xy 157.48 52.07) (xy 168.91 52.07)
 		)
 		(stroke
@@
 	(wire
 		(pts
-			(xy 149.86 53.34) (xy 161.29 53.34)
+			(xy 157.48 62.23) (xy 168.91 62.23)
 		)
 		(stroke
@@
 	(wire
 		(pts
-			(xy 161.29 52.07) (xy 161.29 53.34)
+			(xy 168.91 60.96) (xy 168.91 62.23)
 		)
 		(stroke
@@
 	(wire
 		(pts
-			(xy 161.29 41.91) (xy 161.29 43.18)
-		)
-		(stroke
-			(width 0)
-			(type default)
-		)
-	)
-	(wire
-		(pts
 			(xy 144.78 102.87) (xy 140.97 102.87)
 		)
@@
 	(wire
 		(pts
-			(xy 161.29 53.34) (xy 161.29 54.61)
+			(xy 168.91 62.23) (xy 168.91 63.5)
 		)
 		(stroke
@@
 	(wire
 		(pts
-			(xy 149.86 44.45) (xy 149.86 43.18)
+			(xy 157.48 53.34) (xy 157.48 52.07)
 		)
 		(stroke
@@
 	(wire
 		(pts
-			(xy 161.29 53.34) (xy 172.72 53.34)
+			(xy 168.91 62.23) (xy 180.34 62.23)
 		)
 		(stroke
@@
 	(wire
 		(pts
-			(xy 149.86 52.07) (xy 149.86 53.34)
+			(xy 157.48 60.96) (xy 157.48 62.23)
 		)
 		(stroke
@@
 		)
 	)
-	(hierarchical_label "+3V3"
-		(shape passive)
-		(at 161.29 41.91 90)
-		(effects
-			(font
-				(size 1.27 1.27)
-			)
-			(justify left)
-		)
-	)
 	(hierarchical_label "GND"
 		(shape passive)
@@
 	(symbol
 		(lib_id "power:GND")
-		(at 161.29 54.61 0)
+		(at 168.91 63.5 0)
 		(unit 1)
 		(exclude_from_sim no)
@@
 		(dnp no)
 		(fields_autoplaced yes)
-		(property "Reference" "#PWR026"
-			(at 161.29 60.96 0)
+		(property "Reference" "#PWR017"
+			(at 168.91 69.85 0)
 			(effects
 				(font
@@
 		)
 		(property "Value" "GND"
-			(at 161.29 59.69 0)
+			(at 168.91 68.58 0)
 			(effects
 				(font
@@
 		)
 		(property "Footprint" ""
-			(at 161.29 54.61 0)
+			(at 168.91 63.5 0)
 			(effects
 				(font
@@
 		)
 		(property "Datasheet" ""
-			(at 161.29 54.61 0)
+			(at 168.91 63.5 0)
 			(effects
 				(font
@@
 		)
 		(property "Description" "Power symbol creates a global label with name \"GND\" , ground"
-			(at 161.29 54.61 0)
+			(at 168.91 63.5 0)
 			(effects
 				(font
@@
 			(project "Timing Card"
 				(path "/b0fb402c-3ef3-47ab-87a7-c9cf76e376c0/6789c53e-f0d5-4d0b-a10f-2e5d138a4762"
-					(reference "#PWR026")
+					(reference "#PWR017")
 					(unit 1)
 				)
@@
 		(dnp no)
 		(fields_autoplaced yes)
-		(property "Reference" "#PWR023"
+		(property "Reference" "#PWR015"
 			(at 102.87 142.24 0)
 			(effects
@@
 			(project "Timing Card"
 				(path "/b0fb402c-3ef3-47ab-87a7-c9cf76e376c0/6789c53e-f0d5-4d0b-a10f-2e5d138a4762"
-					(reference "#PWR023")
+					(reference "#PWR015")
 					(unit 1)
 				)
@@
 		(dnp no)
 		(fields_autoplaced yes)
-		(property "Reference" "J10"
+		(property "Reference" "J8"
 			(at 128.27 44.45 0)
 			(effects
@@
 			(project "Instrumentation Control R1"
 				(path "/b0fb402c-3ef3-47ab-87a7-c9cf76e376c0/6789c53e-f0d5-4d0b-a10f-2e5d138a4762"
-					(reference "J10")
+					(reference "J8")
 					(unit 1)
 				)
@@
 	(symbol
 		(lib_id "Device:C")
-		(at 172.72 48.26 0)
+		(at 180.34 57.15 0)
 		(unit 1)
 		(exclude_from_sim no)
@@
 		(on_board yes)
 		(dnp no)
-		(property "Reference" "C90"
-			(at 176.53 46.9899 0)
+		(property "Reference" "C3"
+			(at 184.15 55.8799 0)
 			(effects
 				(font
@@
 		)
 		(property "Value" "10uF"
-			(at 176.53 49.5299 0)
+			(at 184.15 58.4199 0)
 			(effects
 				(font
@@
 		)
 		(property "Footprint" "Capacitor_SMD:CP_Elec_6.3x5.9"
-			(at 173.6852 52.07 0)
+			(at 181.3052 60.96 0)
 			(effects
 				(font
@@
 		)
 		(property "Datasheet" "~"
-			(at 172.72 48.26 0)
+			(at 180.34 57.15 0)
 			(effects
 				(font
@@
 		)
 		(property "Description" "Unpolarized capacitor"
-			(at 172.72 48.26 0)
+			(at 180.34 57.15 0)
 			(effects
 				(font
@@
 			(project "Instrumentation Control R1"
 				(path "/b0fb402c-3ef3-47ab-87a7-c9cf76e376c0/6789c53e-f0d5-4d0b-a10f-2e5d138a4762"
-					(reference "C90")
+					(reference "C3")
 					(unit 1)
 				)
@@
 		(dnp no)
 		(fields_autoplaced yes)
-		(property "Reference" "#PWR027"
+		(property "Reference" "#PWR016"
 			(at 153.67 142.24 0)
 			(effects
@@
 			(project "Timing Card"
 				(path "/b0fb402c-3ef3-47ab-87a7-c9cf76e376c0/6789c53e-f0d5-4d0b-a10f-2e5d138a4762"
-					(reference "#PWR027")
+					(reference "#PWR016")
 					(unit 1)
 				)
@@
 	(symbol
 		(lib_id "Device:C")
-		(at 161.29 48.26 0)
+		(at 168.91 57.15 0)
 		(unit 1)
 		(exclude_from_sim no)
@@
 		(dnp no)
 		(fields_autoplaced yes)
-		(property "Reference" "C89"
-			(at 165.1 46.9899 0)
+		(property "Reference" "C2"
+			(at 172.72 55.8799 0)
 			(effects
 				(font
@@
 		)
 		(property "Value" "1uF"
-			(at 165.1 49.5299 0)
+			(at 172.72 58.4199 0)
 			(effects
 				(font
@@
 		)
 		(property "Footprint" "Capacitor_SMD:C_0603_1608Metric"
-			(at 162.2552 52.07 0)
+			(at 169.8752 60.96 0)
 			(effects
 				(font
@@
 		)
 		(property "Datasheet" "~"
-			(at 161.29 48.26 0)
+			(at 168.91 57.15 0)
 			(effects
 				(font
@@
 		)
 		(property "Description" "Unpolarized capacitor"
-			(at 161.29 48.26 0)
+			(at 168.91 57.15 0)
 			(effects
 				(font
@@
 			(project "Instrumentation Control R1"
 				(path "/b0fb402c-3ef3-47ab-87a7-c9cf76e376c0/6789c53e-f0d5-4d0b-a10f-2e5d138a4762"
-					(reference "C89")
+					(reference "C2")
 					(unit 1)
 				)
@@
 	(symbol
 		(lib_id "Device:C")
-		(at 149.86 48.26 0)
+		(at 157.48 57.15 0)
 		(unit 1)
 		(exclude_from_sim no)
@@
 		(on_board yes)
 		(dnp no)
-		(property "Reference" "C88"
-			(at 153.67 46.9899 0)
+		(property "Reference" "C1"
+			(at 161.29 55.8799 0)
 			(effects
 				(font
@@
 		)
 		(property "Value" "0.1uF"
-			(at 153.67 49.5299 0)
+			(at 161.29 58.4199 0)
 			(effects
 				(font
@@
 		)
 		(property "Footprint" "Capacitor_SMD:C_0603_1608Metric"
-			(at 150.8252 52.07 0)
+			(at 158.4452 60.96 0)
 			(effects
 				(font
@@
 		)
 		(property "Datasheet" "~"
-			(at 149.86 48.26 0)
+			(at 157.48 57.15 0)
 			(effects
 				(font
@@
 		)
 		(property "Description" "Unpolarized capacitor"
-			(at 149.86 48.26 0)
+			(at 157.48 57.15 0)
 			(effects
 				(font
@@
 			(project "Instrumentation Control R1"
 				(path "/b0fb402c-3ef3-47ab-87a7-c9cf76e376c0/6789c53e-f0d5-4d0b-a10f-2e5d138a4762"
-					(reference "C88")
+					(reference "C1")
 					(unit 1)
 				)

Commit message: Camera Control Card layout
Parts:
- C1, C2: footprint Capacitor_SMD:C_0603_1608Metric -> Capacitor_SMD:C_0805_2012Metric
Changed lines of the file:
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@@
 			)
 		)
-		(property "Footprint" "Capacitor_SMD:C_0603_1608Metric"
+		(property "Footprint" "Capacitor_SMD:C_0805_2012Metric"
 			(at 169.8752 60.96 0)
 			(effects
@@
 			)
 		)
-		(property "Footprint" "Capacitor_SMD:C_0603_1608Metric"
+		(property "Footprint" "Capacitor_SMD:C_0805_2012Metric"
 			(at 158.4452 60.96 0)
 			(effects
