File: Camera-Control-Card/Tristate.kicad_sch (KiCad schematic)
At the start: 2 parts, among them U2 SN74LVC1G125DRL

Commit message: test
Parts:
- C6: footprint Capacitor_SMD:C_0805_2012Metric -> Capacitor_SMD:C_0603_1608Metric
Changed lines of the file:
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@@
 			)
 		)
-		(property "Footprint" "Capacitor_SMD:C_0805_2012Metric"
+		(property "Footprint" "Capacitor_SMD:C_0603_1608Metric"
 			(at 133.6548 95.25 0)
 			(effects

Commit message: Updates
Parts:
- renumbered C6 to C42, U2 to U3
Changed lines of the file:
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@@
 		(on_board yes)
 		(dnp no)
-		(property "Reference" "#PWR0102"
+		(property "Reference" "#PWR063"
 			(at 139.7 121.92 0)
 			(effects
@@
 			(project "Timing Card"
 				(path "/b0fb402c-3ef3-47ab-87a7-c9cf76e376c0/ae4f5bb6-a0ce-4bcc-8790-572e089af1bb/63a1c871-f7c8-40c9-a25d-fb41c3b6e016"
-					(reference "#PWR0102")
+					(reference "#PWR063")
 					(unit 1)
 				)
@@
 		(on_board yes)
 		(dnp no)
-		(property "Reference" "U2"
+		(property "Reference" "U3"
 			(at 144.272 107.696 0)
 			(effects
@@
 			(project "Pump Control Card R1"
 				(path "/b0fb402c-3ef3-47ab-87a7-c9cf76e376c0/ae4f5bb6-a0ce-4bcc-8790-572e089af1bb/63a1c871-f7c8-40c9-a25d-fb41c3b6e016"
-					(reference "U2")
+					(reference "U3")
 					(unit 1)
 				)
@@
 		(on_board yes)
 		(dnp no)
-		(property "Reference" "#PWR0103"
+		(property "Reference" "#PWR061"
 			(at 134.62 102.87 0)
 			(effects
@@
 			(project "Timing Card"
 				(path "/b0fb402c-3ef3-47ab-87a7-c9cf76e376c0/ae4f5bb6-a0ce-4bcc-8790-572e089af1bb/63a1c871-f7c8-40c9-a25d-fb41c3b6e016"
-					(reference "#PWR0103")
+					(reference "#PWR061")
 					(unit 1)
 				)
@@
 		(on_board yes)
 		(dnp no)
-		(property "Reference" "C6"
+		(property "Reference" "C42"
 			(at 134.366 89.408 0)
 			(effects
@@
 			(project "Timing Card"
 				(path "/b0fb402c-3ef3-47ab-87a7-c9cf76e376c0/ae4f5bb6-a0ce-4bcc-8790-572e089af1bb/63a1c871-f7c8-40c9-a25d-fb41c3b6e016"
-					(reference "C6")
+					(reference "C42")
 					(unit 1)
 				)
@@
 		(on_board yes)
 		(dnp no)
-		(property "Reference" "#PWR0101"
+		(property "Reference" "#PWR062"
 			(at 139.7 88.9 0)
 			(effects
@@
 			(project "Timing Card"
 				(path "/b0fb402c-3ef3-47ab-87a7-c9cf76e376c0/ae4f5bb6-a0ce-4bcc-8790-572e089af1bb/63a1c871-f7c8-40c9-a25d-fb41c3b6e016"
-					(reference "#PWR0101")
-					(unit 1)
-				)
+					(reference "#PWR062")
+					(unit 1)
+				)
