File: Camera-Control-Card/Buffer_3V3.kicad_sch (KiCad schematic)
At the start: 11 parts, among them U3 74AHC125

Commit message: test
Parts:
- removed R19: 10K, symbol Device:R
- removed R20: 22R, symbol Device:R
- added C5: 1uF, Capacitor_SMD:C_0603_1608Metric, symbol Device:C
- added C7: 0.1uF, Capacitor_SMD:C_0603_1608Metric, symbol Device:C
- added D1, D13, D17, D2, D4: R, Resistor_SMD:R_0603_1608Metric, symbol Device:LED
- added D10, D12, D16, D19, D5: 3V3, Diode_SMD:D_SOD-323, symbol Device:D_Zener
- added R21, R23, R24, R31, R37: 1K, Resistor_SMD:R_0603_1608Metric, symbol Device:R
- added R29, R35: 10K, Resistor_SMD:R_0603_1608Metric, symbol Device:R
- added R34, R39: 22R, Resistor_SMD:R_0603_1608Metric, symbol Device:R
- added U4: 74AHC125, Package_SO:TSSOP-14_4.4x5mm_P0.65mm, symbol 74xx:74AHCT125
- C3, C4: footprint (none) -> Capacitor_SMD:C_0603_1608Metric
- R13, R14, R15, R16, R17, R18: footprint (none) -> Resistor_SMD:R_0603_1608Metric
Connections:
- net OUT_3 is gone; now on net OUT_2: R16.2
- net +3V3: now also U3.10, C5.1, C7.1, R29.1, R35.1, U4.10, U4.13, U4.14 (VCC)
- net GND: now also U3.9, C5.2, C7.2, D1.1 (K), D10.2 (A), D12.2 (A), D13.1 (K), D16.2 (A), D17.1 (K), D19.2 (A), D2.1 (K), D4.1 (K), D5.2 (A), U4.12, U4.7 (GND), U4.9
- net IN_2: now also U3.12; no longer U3.9
- net IN_3: now also U4.2; no longer U3.12
- net OE_2: now also R14.2, U3.13; no longer U3.10
- net OE_3: now also R29.2, U4.1; no longer R14.2, U3.13
- net OUT_0: now also D5.1 (K)
- net OUT_1: now also D10.1 (K)
- net OUT_2: now also D12.1 (K), D16.1 (K), R34.2
- net at R16.1, U3.11: now also R24.2
- net at R18.1, U3.6: now also R23.2
- net at R15.1, U3.3: now also R21.2
- new net: D17.2 (A), R37.1
- new net: D4.2 (A), R24.1
- new net: R37.2, R39.1, U4.6
- new net: D13.2 (A), R31.1
- new net: R31.2, R34.1, U4.3
- new net: D1.2 (A), R21.1
- new net: D2.2 (A), R23.1
- new net IN_4: U4.5
- new net OE_4: R35.2, U4.4
- new net OUT_4: D19.1 (K), R39.2
- no-connect marks 0 -> 3
Other:
- moved on the sheet: C3, C4, R13, R14, R15, R16, R17, R18, U3A, U3B, U3C, U3D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

Commit message: Updates
Parts:
- D10: renamed from D12; value 3V3 -> D_3V3
- D11: renamed from D13; footprint Resistor_SMD:R_0603_1608Metric -> LED_SMD:LED_0603_1608Metric
- D12: renamed from D16; value 3V3 -> D_3V3
- D13: renamed from D17; footprint Resistor_SMD:R_0603_1608Metric -> LED_SMD:LED_0603_1608Metric
- D14: renamed from D19; value 3V3 -> D_3V3
- D5: renamed from D1; footprint Resistor_SMD:R_0603_1608Metric -> LED_SMD:LED_0603_1608Metric
- D6: renamed from D5; value 3V3 -> D_3V3
- D7: renamed from D2; footprint Resistor_SMD:R_0603_1608Metric -> LED_SMD:LED_0603_1608Metric
- D8: renamed from D4; footprint Resistor_SMD:R_0603_1608Metric -> LED_SMD:LED_0603_1608Metric
- D9: renamed from D10; value 3V3 -> D_3V3
- renumbered C3 to C43, C4 to C44, C5 to C45, C7 to C46, R13 to R17, R21 to R18, R15 to R19, R17 to R20, R14 to R21, R23 to R22, R24 to R23, R18 to R24, R16 to R25, R29 to R26, R31 to R27, R34 to R28, R35 to R29, R37 to R30, R39 to R31, U3 to U4, U4 to U5
Connections:
- net IN_0: now also U4.5; no longer U4.2
- net IN_1: now also U4.2; no longer U4.5
- net OE_0: now also R20.2, U4.4; no longer R17.2, U4.1
- net OE_1: now also R17.2, U4.1; no longer R20.2, U4.4
- net OUT_0: now also D9.1 (K), R24.2; no longer D6.1 (K), R19.2
- net OUT_1: now also D6.1 (K), R19.2; no longer D9.1 (K), R24.2
- net OUT_2: no longer D12.1 (K), R28.2
- new net OUT_3: D12.1 (K), R28.2

Commit message: Layout completed for camera control card
Connections:
- net +3V3: now also U5.4; no longer U5.13
- net GND: now also U5.5; no longer U5.12
- net IN_4: now also U5.12; no longer U5.5
- net OE_4: now also U5.13; no longer U5.4
- net at R30.2, R31.1: now also U5.11; no longer U5.6
