File: Camera-Control-Card/Camera-Control-Card.kicad_pcb (KiCad board)
At the start: 2 copper layers, 65 x 41.6 mm, 74 parts, among them J10 10018784-10201TLF, J2 Conn_01x10, U1 LCMXO2-7000HC-6TG144I, U11 T602-025.0M, U2 SN74LVC1G125DRL, U3 74AHC125

Commit message: test
Parts:
- removed C91: 0.1uF, Capacitor_SMD:C_0805_2012Metric
- removed C93: 1uF, Capacitor_SMD:C_0805_2012Metric
- removed C96: 10uF, Capacitor_SMD:CP_Elec_6.3x5.9
- removed TP10, TP11, TP12, TP13, TP14, TP15, TP7, TP8, TP9: TestPoint, TestPoint:TestPoint_Pad_1.0x1.0mm
- added C3: 1uF, Capacitor_SMD:C_0603_1608Metric, F.Cu at (201.6, 66.0)
- added C4: 0.1uF, Capacitor_SMD:C_0603_1608Metric, F.Cu at (201.6, 68.5)
- added C5: 1uF, Capacitor_SMD:C_0603_1608Metric, F.Cu at (228.2, 63.9)
- added C7: 0.1uF, Capacitor_SMD:C_0603_1608Metric, F.Cu at (228.2, 66.4)
- added D1: R, Resistor_SMD:R_0603_1608Metric, F.Cu at (201.6, 71.0)
- added D10: 3V3, Diode_SMD:D_SOD-323, F.Cu at (241.1, 42.5)
- added D12: 3V3, Diode_SMD:D_SOD-323, F.Cu at (241.1, 45.4)
- added D13: R, Resistor_SMD:R_0603_1608Metric, F.Cu at (228.2, 68.9)
- added D16: 3V3, Diode_SMD:D_SOD-323, F.Cu at (241.1, 51.3)
- added D17: R, Resistor_SMD:R_0603_1608Metric, F.Cu at (228.2, 73.9)
- added D19: 3V3, Diode_SMD:D_SOD-323, F.Cu at (241.1, 54.3)
- added D2: R, Resistor_SMD:R_0603_1608Metric, F.Cu at (201.6, 73.5)
- added D4: R, Resistor_SMD:R_0603_1608Metric, F.Cu at (201.6, 78.5)
- added D5: 3V3, Diode_SMD:D_SOD-323, F.Cu at (241.1, 39.5)
- added D6: B, Resistor_SMD:R_0603_1608Metric, F.Cu at (195.2, 63.4)
- added D7: B, Resistor_SMD:R_0603_1608Metric, F.Cu at (195.2, 65.9)
- added D8: B, Resistor_SMD:R_0603_1608Metric, F.Cu at (195.2, 68.5)
- added D9: B, Resistor_SMD:R_0603_1608Metric, F.Cu at (195.2, 71.0)
- added J1: Conn_Coaxial, Connector_Coaxial:SMA_Molex_73251-1153_EdgeMount_Horizontal, F.Cu at (127.5, 83.2)
- added J3: Conn_Coaxial, Connector_Coaxial:SMA_Molex_73251-1153_EdgeMount_Horizontal, F.Cu at (152.5, 83.2)
- added J4: Conn_Coaxial, Connector_Coaxial:SMA_Molex_73251-1153_EdgeMount_Horizontal, F.Cu at (165.0, 83.2)
- added J5: Conn_Coaxial, Connector_Coaxial:SMA_Molex_73251-1153_EdgeMount_Horizontal, F.Cu at (177.5, 83.2)
- added J7: Conn_01x10, Footprints:AMPHENOL_78207-110HLF, F.Cu at (133.0, 111.5)
- added J8: SFV24R-1STE1HLF, Footprints:AMPHENOL_SFV24R-1STE1HLF, F.Cu at (123.5, 95.5)
- added R13: 10K, Resistor_SMD:R_0603_1608Metric, F.Cu at (201.6, 81.0)
- added R14: 10K, Resistor_SMD:R_0603_1608Metric, F.Cu at (205.6, 66.0)
- added R15: 22R, Resistor_SMD:R_0603_1608Metric, F.Cu at (205.6, 68.5)
- added R16: 22R, Resistor_SMD:R_0603_1608Metric, F.Cu at (205.6, 71.0)
- added R17: 10K, Resistor_SMD:R_0603_1608Metric, F.Cu at (205.6, 73.5)
- added R18: 22R, Resistor_SMD:R_0603_1608Metric, F.Cu at (205.6, 76.0)
- added R21: 1K, Resistor_SMD:R_0603_1608Metric, F.Cu at (209.6, 66.0)
- added R23: 1K, Resistor_SMD:R_0603_1608Metric, F.Cu at (209.6, 71.0)
- added R24: 1K, Resistor_SMD:R_0603_1608Metric, F.Cu at (209.6, 73.5)
- added R25: 1K, Resistor_SMD:R_0603_1608Metric, F.Cu at (195.2, 73.5)
- added R26: 1K, Resistor_SMD:R_0603_1608Metric, F.Cu at (195.2, 76.0)
- added R27: 1K, Resistor_SMD:R_0603_1608Metric, F.Cu at (195.2, 78.5)
- added R28: 1K, Resistor_SMD:R_0603_1608Metric, F.Cu at (195.2, 81.0)
- added R29: 10K, Resistor_SMD:R_0603_1608Metric, F.Cu at (228.2, 78.9)
- added R31: 1K, Resistor_SMD:R_0603_1608Metric, F.Cu at (232.2, 66.4)
- added R34: 22R, Resistor_SMD:R_0603_1608Metric, F.Cu at (232.2, 73.9)
- added R35: 10K, Resistor_SMD:R_0603_1608Metric, F.Cu at (232.2, 76.4)
- added R37: 1K, Resistor_SMD:R_0603_1608Metric, F.Cu at (236.3, 63.9)
- added R39: 22R, Resistor_SMD:R_0603_1608Metric, F.Cu at (236.3, 68.9)
- added U4: 74AHC125, Package_SO:TSSOP-14_4.4x5mm_P0.65mm, F.Cu at (242.6, 66.0)
- C1, C2, C6, C88, C89: footprint Capacitor_SMD:C_0805_2012Metric -> Capacitor_SMD:C_0603_1608Metric
- J2: value Conn_01x10 -> Conn_Coaxial; footprint Connector_PinHeader_2.54mm:PinHeader_2x05_P2.54mm_Vertical -> Connector_Coaxial:SMA_Molex_73251-1153_EdgeMount_Horizontal
- moved J2 96.0 mm to (140.0, 83.2), turned to -90 degrees
- moved U1 75.8 mm to (151.5, 102.0), turned to 90 degrees
- moved U3 58.4 mm to (216.0, 68.1)
- moved U11 17.5 mm to (218.6, 93.7)
Connections:
- C57 pad 1: +3V3 -> GND
- C58 pad 1: +3V3 -> GND
- J10 pad A10: /PCIe/+5V -> unconnected-(J10-PadA10)
- J10 pad A11: /PCIe/+5V -> unconnected-(J10-PadA11)
- J10 pad A12: /PCIe/+5V -> unconnected-(J10-PadA12)
- J10 pad A13: /PCIe/+5V -> unconnected-(J10-PadA13)
- J10 pad A14: /PCIe/+5V -> unconnected-(J10-PadA14)
- J10 pad A15: /PCIe/+5V -> unconnected-(J10-PadA15)
- J10 pad A9: /PCIe/+5V -> unconnected-(J10-PadA9)
- J2 pad 1: GND -> /Buffer_3V3/OUT_1
- J2 pad 2: +3V3 -> GND
- U1 pad 1: Net-(U1A-PL3A) -> unconnected-(U1A-PL3A-Pad1)
- U1 pad 10: Net-(U1A-PL8B) -> unconnected-(U1A-PL8B-Pad10)
- U1 pad 14: Net-(U1A-PL10B) -> unconnected-(U1A-PL10B-Pad14)
- U1 pad 19: Net-(U1A-PL12A) -> unconnected-(U1A-PL12A-Pad19)
- U1 pad 23: Net-(U1A-PL17A) -> unconnected-(U1A-PL17A-Pad23)
- U1 pad 27: Net-(U1A-PL22A) -> unconnected-(U1A-PL22A-Pad27)
- U1 pad 31: Net-(U1A-PL23D) -> unconnected-(U1A-PL23D-Pad31)
- U1 pad 35: Net-(U1A-PL25B) -> unconnected-(U1A-PL25B-Pad35)
- U1 pad 6: Net-(U1A-PL6B) -> unconnected-(U1A-PL6B-Pad6)
- U3 pad 1: unconnected-(U3-Pad1) -> /Buffer_3V3/OE_0
- U3 pad 10: unconnected-(U3-Pad10) -> +3V3
- U3 pad 11: unconnected-(U3-Pad11) -> Net-(R16-Pad1)
- U3 pad 12: unconnected-(U3-Pad12) -> /Buffer_3V3/IN_2
- U3 pad 13: unconnected-(U3-Pad13) -> /Buffer_3V3/OE_2
- U3 pad 2: unconnected-(U3-Pad2) -> /Buffer_3V3/IN_0
- U3 pad 3: unconnected-(U3-Pad3) -> Net-(R15-Pad1)
- U3 pad 4: unconnected-(U3-Pad4) -> /Buffer_3V3/OE_1
- U3 pad 5: unconnected-(U3-Pad5) -> /Buffer_3V3/IN_1
- U3 pad 6: unconnected-(U3-Pad6) -> Net-(R18-Pad1)
- U3 pad 7: unconnected-(U3E-GND-Pad7) -> GND
- U3 pad 9: unconnected-(U3-Pad9) -> GND
Routing:
- added copper zone on B.Cu, net GND
- added copper zone on In1.Cu, net GND
Other:
- copper layers 2 -> 4

Commit message: Updates
Parts:
- removed the J7 at (133.0, 111.5)
- added C47: 1uF, Capacitor_SMD:C_0603_1608Metric, F.Cu at (177.9, 93.4)
- added C48: 0.1uF, Capacitor_SMD:C_0603_1608Metric, F.Cu at (174.1, 97.7)
- added C49: 4.7uF, Capacitor_SMD:C_0603_1608Metric, F.Cu at (175.6, 97.7)
- added C50: 0.1uF, Capacitor_SMD:C_0603_1608Metric, F.Cu at (174.1, 94.7)
- added C51: 4.7uF, Capacitor_SMD:C_0603_1608Metric, F.Cu at (172.6, 96.3)
- added D15: D_5V, Diode_SMD:D_SOD-323, F.Cu at (188.9, 90.5)
- added D16: B, LED_SMD:LED_0603_1608Metric, F.Cu at (180.0, 112.0)
- added F1: Fuse, Fuse:Fuse_0603_1608Metric, F.Cu at (175.6, 94.7)
- added J2: Conn_02x05_Counter_Clockwise, Footprints:AMPHENOL_78207-110HLF, F.Cu at (133.0, 111.5)
- added J9: USB_C_Receptacle_USB2.0_16P, Connector_USB:USB_C_Receptacle_G-Switch_GT-USB-7010ASV, F.Cu at (181.2, 99.5)
- added R32: 5.1K, Resistor_SMD:R_0603_1608Metric, F.Cu at (164.7, 44.5)
- added R33: 5.1K, Resistor_SMD:R_0603_1608Metric, F.Cu at (164.2, 49.5)
- added R34: 22.1K, Resistor_SMD:R_0603_1608Metric, F.Cu at (171.8, 94.0)
- added R35: 47.5K, Resistor_SMD:R_0603_1608Metric, F.Cu at (170.3, 95.5)
- added R36: 1K, Resistor_SMD:R_0603_1608Metric, F.Cu at (169.7, 97.0)
- added R37: 1K, Resistor_SMD:R_0603_1608Metric, F.Cu at (180.0, 109.0)
- added U6: TPD2EUSB30, Package_TO_SOT_SMD:Texas_DRT-3, F.Cu at (156.5, 54.8)
- added U7: CP2102N-Axx-xQFN20, Package_DFN_QFN:SiliconLabs_QFN-20-1EP_3x3mm_P0.5mm_EP1.8x1.8mm, F.Cu at (171.0, 100.0)
- D1: renamed from D6; footprint Resistor_SMD:R_0603_1608Metric -> LED_SMD:LED_0603_1608Metric
- D10: renamed from D12; value 3V3 -> D_3V3
- D11: renamed from D13; footprint Resistor_SMD:R_0603_1608Metric -> LED_SMD:LED_0603_1608Metric
- D12: renamed from D16; value 3V3 -> D_3V3
- D13: renamed from D17; footprint Resistor_SMD:R_0603_1608Metric -> LED_SMD:LED_0603_1608Metric
- D14: renamed from D19; value 3V3 -> D_3V3
- D2: renamed from D7; footprint Resistor_SMD:R_0603_1608Metric -> LED_SMD:LED_0603_1608Metric
- D3: renamed from D8; footprint Resistor_SMD:R_0603_1608Metric -> LED_SMD:LED_0603_1608Metric
- D4: renamed from D9; footprint Resistor_SMD:R_0603_1608Metric -> LED_SMD:LED_0603_1608Metric
- D5: renamed from D1; footprint Resistor_SMD:R_0603_1608Metric -> LED_SMD:LED_0603_1608Metric
- D6: renamed from D5; value 3V3 -> D_3V3
- D7: renamed from D2; footprint Resistor_SMD:R_0603_1608Metric -> LED_SMD:LED_0603_1608Metric
- D8: renamed from D4; footprint Resistor_SMD:R_0603_1608Metric -> LED_SMD:LED_0603_1608Metric
- D9: renamed from D10; value 3V3 -> D_3V3
- R1: renamed from R4; footprint Resistor_SMD:R_0805_2012Metric -> Resistor_SMD:R_0603_1608Metric
- R10: renamed from R7; footprint Resistor_SMD:R_0805_2012Metric -> Resistor_SMD:R_0603_1608Metric
- R11: renamed from R8; footprint Resistor_SMD:R_0805_2012Metric -> Resistor_SMD:R_0603_1608Metric
- R12: renamed from R11; footprint Resistor_SMD:R_0805_2012Metric -> Resistor_SMD:R_0603_1608Metric
- R2: renamed from R1; footprint Resistor_SMD:R_0805_2012Metric -> Resistor_SMD:R_0603_1608Metric
- R3: renamed from R2; footprint Resistor_SMD:R_0805_2012Metric -> Resistor_SMD:R_0603_1608Metric
- R4: renamed from R3; footprint Resistor_SMD:R_0805_2012Metric -> Resistor_SMD:R_0603_1608Metric
- R5: renamed from R9; footprint Resistor_SMD:R_0805_2012Metric -> Resistor_SMD:R_0603_1608Metric
- R6: renamed from R10; footprint Resistor_SMD:R_0805_2012Metric -> Resistor_SMD:R_0603_1608Metric
- R7: renamed from R12; footprint Resistor_SMD:R_0805_2012Metric -> Resistor_SMD:R_0603_1608Metric
- R8: renamed from R5; footprint Resistor_SMD:R_0805_2012Metric -> Resistor_SMD:R_0603_1608Metric
- R9: renamed from R6; footprint Resistor_SMD:R_0805_2012Metric -> Resistor_SMD:R_0603_1608Metric
- moved R22 81.6 mm to (129.9, 88.2)
- moved R24 76.5 mm to (129.9, 86.7), turned to 180 degrees
- moved R2 76.4 mm to (136.5, 140.7), turned to 180 degrees
- moved D7 75.3 mm to (127.6, 87.5), turned to -90 degrees
- moved U5 74.8 mm to (171.3, 88.7)
- moved R18 73.7 mm to (139.4, 88.2)
- moved R10 72.9 mm to (144.5, 146.9)
- moved R11 72.9 mm to (144.5, 149.8)
- moved R8 72.9 mm to (144.5, 141.0)
- moved R9 72.9 mm to (144.5, 143.9)
- moved U4 72.7 mm to (146.3, 88.7)
- moved R3 72.3 mm to (140.5, 141.4), turned to 180 degrees
- moved R4 71.4 mm to (141.7, 135.4)
- moved R27 71.3 mm to (164.4, 88.2)
- moved R28 69.0 mm to (164.4, 86.7), turned to 180 degrees
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- renumbered C88 to C1, C33 to C10, C40 to C11, C41 to C12, C35 to C13, C36 to C14, C38 to C15, C42 to C16, C34 to C17, C37 to C18, C39 to C19, C89 to C2, C43 to C20, C45 to C21, C52 to C22, C46 to C23, C48 to C24, C50 to C25, C53 to C26, C47 to C27, C49 to C28, C51 to C29, C90 to C3, C54 to C30, C1 to C31, C2 to C32, C61 to C33, C55 to C34, C57 to C35, C59 to C36, C62 to C37, C56 to C38, C58 to C39, C28 to C4, C60 to C40, C63 to C41, C6 to C42, C3 to C43, C4 to C44, C5 to C45, C7 to C46, C30 to C5, C32 to C6, C44 to C7, C29 to C8, C31 to C9, J8 to J1, J1 to J3, J2 to J4, J3 to J5, J4 to J6, J5 to J7, J10 to J8, R25 to R13, R26 to R14, R27 to R15, R28 to R16, R13 to R17, R21 to R18, R15 to R19, R17 to R20, R14 to R21, R23 to R22, R24 to R23, R18 to R24, R16 to R25, R29 to R26, R31 to R27, R34 to R28, R35 to R29, R37 to R30, R39 to R31, TP19 to TP1, U11 to U2, U2 to U3, U3 to U4, U4 to U5
Connections:
- net /FPGA/DONE renamed /DONE
- net /FPGA/INITN renamed /INIT_N
- net /FPGA/PROGRAMN renamed /PROGRAMN
- net /FPGA/TCK renamed /TCK
- net /FPGA/TDI renamed /TDI
- net /FPGA/TDO renamed /TDO
- net /FPGA/TMS renamed /TMS
- D10 pad 1: /Buffer_3V3/OUT_3 -> /Buffer_3V3/OUT_2
- D6 pad 1: /Buffer_3V3/OUT_0 -> /Buffer_3V3/OUT_1
- D9 pad 1: /Buffer_3V3/OUT_1 -> /Buffer_3V3/OUT_0
- J1 pad 1: unconnected-(J8-Pad1) -> /FPGA/PT35B
- J1 pad 11: unconnected-(J8-Pad11) -> /FPGA/PT28A
- J1 pad 13: unconnected-(J8-Pad13) -> /FPGA/PT25B
- J1 pad 15: unconnected-(J8-Pad15) -> /FPGA/PT25A
- J1 pad 17: unconnected-(J8-Pad17) -> /FPGA/PT22D
- J1 pad 19: unconnected-(J8-Pad19) -> /FPGA/PT22C
- J1 pad 21: unconnected-(J8-Pad21) -> /FPGA/PT18B
- J1 pad 23: unconnected-(J8-Pad23) -> /FPGA/PT18A
- J1 pad 3: unconnected-(J8-Pad3) -> /FPGA/PT35A
- J1 pad 5: unconnected-(J8-Pad5) -> /FPGA/PT33B
- J1 pad 7: unconnected-(J8-Pad7) -> /FPGA/PT33A
- J1 pad 9: unconnected-(J8-Pad9) -> /FPGA/PT28B
- J5 pad 1: /Buffer_3V3/OUT_3 -> /Buffer_3V3/OUT_2
- R17 pad 2: /Buffer_3V3/OE_0 -> /Buffer_3V3/OE_1
- R19 pad 2: /Buffer_3V3/OUT_0 -> /Buffer_3V3/OUT_1
- R20 pad 2: /Buffer_3V3/OE_1 -> /Buffer_3V3/OE_0
- R24 pad 2: /Buffer_3V3/OUT_1 -> /Buffer_3V3/OUT_0
- R25 pad 2: /Buffer_3V3/OUT_3 -> /Buffer_3V3/OUT_2
- U1 pad 111: unconnected-(U1B-PT35B-Pad111) -> /FPGA/PT35B
- U1 pad 112: unconnected-(U1B-PT35A-Pad112) -> /FPGA/PT35A
- U1 pad 113: unconnected-(U1B-PT33B-Pad113) -> /FPGA/PT33B
- U1 pad 114: unconnected-(U1B-PT33A-Pad114) -> /FPGA/PT33A
- U1 pad 115: unconnected-(U1B-PT28B-Pad115) -> /FPGA/PT28B
- U1 pad 117: unconnected-(U1B-PT28A-Pad117) -> /FPGA/PT28A
- U1 pad 121: unconnected-(U1B-PT25B-Pad121) -> /FPGA/PT25B
- U1 pad 122: unconnected-(U1B-PT25A-Pad122) -> /FPGA/PT25A
- U1 pad 125: /FPGA/SDA -> /FPGA/PT22D
- U1 pad 126: /FPGA/SCL -> /FPGA/PT22C
- U1 pad 127: unconnected-(U1B-PT18B-Pad127) -> /FPGA/PT18B
- U1 pad 128: /FPGA/OSC_OUT -> /FPGA/PT18A
- U4 pad 1: /Buffer_3V3/OE_0 -> /Buffer_3V3/OE_1
- U4 pad 2: /Buffer_3V3/IN_0 -> /Buffer_3V3/IN_1
- U4 pad 4: /Buffer_3V3/OE_1 -> /Buffer_3V3/OE_0
- U4 pad 5: /Buffer_3V3/IN_1 -> /Buffer_3V3/IN_0
Routing:
- net /FPGA/PT35B: track 0.00 -> 18.4 mm
- net /FPGA/PT35A: track 0.00 -> 18.2 mm
- net /FPGA/PT33B: track 0.00 -> 18.0 mm
- net /FPGA/PT25B: track 0.00 -> 18.0 mm
- net /FPGA/PT22D: track 0.00 -> 18.0 mm
- net /FPGA/PT33A: track 0.00 -> 17.8 mm
- net /FPGA/PT22C: track 0.00 -> 17.8 mm
- net /FPGA/PT25A: track 0.00 -> 17.8 mm
- net /FPGA/PT18B: track 0.00 -> 17.6 mm
- net /FPGA/PT28B: track 0.00 -> 17.6 mm
- net /FPGA/PT28A: track 0.00 -> 17.6 mm
- net /FPGA/PT18A: track 0.00 -> 17.4 mm
- net /FPGA/LED_4: track 0.00 -> 16.3 mm
- net /FPGA/LED_3: track 0.00 -> 14.1 mm
- net Net-(R22-Pad2): track 0.00 -> 13.9 mm
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Other:
- outline, holes or cut-outs redrawn

Commit message: Camera Control Card layout
Parts:
- added C52: 0.1uF, Capacitor_SMD:C_0603_1608Metric, F.Cu at (155.0, 117.2)
- added D17: G, LED_SMD:LED_0603_1608Metric, F.Cu at (165.7, 91.8)
- added R40: 22R, Resistor_SMD:R_0603_1608Metric, F.Cu at (152.7, 119.3)
- added TP2: TestPoint, TestPoint:TestPoint_Pad_D1.0mm, F.Cu at (167.5, 99.1)
- added TP3: TestPoint, TestPoint:TestPoint_Pad_D1.0mm, F.Cu at (165.6, 100.5)
- added U8: SN74LVC1G125DRL, Package_TO_SOT_SMD:Texas_R-PDSO-N5_DRL-5, F.Cu at (153.2, 117.2)
- C1, C2: footprint Capacitor_SMD:C_0603_1608Metric -> Capacitor_SMD:C_0805_2012Metric
- C10, C11, C12, C13, C14, C15, C16, C17, C18, C19, C20, C21, C22, C23, C24, C25, C26, C27, C28, C29, C3, C30, C33, C34, C35, C36, C37, C38, C39, C4, C40, C41, C5, C6, C7, C8, C9, D10, D12, D14, D15, D6, D9, R11, R32, R33, U6: moved to B.Cu
- moved U3 85.7 mm to (145.2, 117.2), turned to -90 degrees
- moved C42 83.5 mm to (147.0, 117.2), turned to 90 degrees
- moved R1 82.2 mm to (137.9, 110.8), turned to -90 degrees
- moved C30 81.1 mm to (139.9, 91.4), turned to 90 degrees
- moved R12 80.1 mm to (144.7, 119.3)
- moved C26 78.4 mm to (141.4, 91.4), turned to 90 degrees
- moved C22 75.4 mm to (142.9, 92.0), turned to 90 degrees
- moved C40 75.3 mm to (141.9, 97.9), turned to 90 degrees
- moved C3 74.2 mm to (126.0, 112.0), turned to 90 degrees
- moved R6 74.1 mm to (164.2, 91.8), turned to 90 degrees
- moved C36 72.8 mm to (143.4, 97.9), turned to 90 degrees
- moved C1 72.7 mm to (136.4, 117.9), turned to -90 degrees
- moved C37 72.0 mm to (141.0, 113.1), turned to 180 degrees
- moved C41 71.8 mm to (141.0, 116.1), turned to 180 degrees
- moved C39 71.1 mm to (141.9, 103.1), turned to -90 degrees
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Connections:
- net /FPGA/MISO renamed /FPGA/MISO_1_BUF
- C35 pad 1: GND -> +3V3
- C39 pad 1: GND -> +3V3
- C48 pad 1: +3.3V -> +3V3
- C49 pad 1: +3.3V -> +3V3
- C50 pad 1: +3.3V -> +3V3
- C51 pad 1: +3.3V -> +3V3
- J2 pad 1: +3V3 -> GND
- J2 pad 2: /PROGRAMN -> GND
- J2 pad 3: /INIT_N -> /DONE
- J2 pad 4: GND -> +3V3
- J2 pad 5: GND -> /PROGRAMN
- J2 pad 6: /DONE -> /INIT_N
- J8 pad B11: /FPGA/MCLK/CCLK -> /FPGA/SCK_1
- J8 pad B12: /FPGA/SI/SISPI -> /FPGA/MOSI_1
- J8 pad B19: /PCIe/SCK_2 -> /FPGA/SCK_2
- J8 pad B20: /PCIe/MOSI_2 -> /FPGA/MOSI_2
- J8 pad B21: /PCIe/MISO_2 -> /FPGA/MISO_2_BUF
- R36 pad 1: +3.3V -> +3V3
- R6 pad 1: +3V3 -> Net-(D17-A)
- R6 pad 2: /FPGA/MCLK/CCLK -> +3V3
- TP1 pad 1: /FPGA/SN -> Net-(U1A-PB35A)
- U1 pad 1: unconnected-(U1A-PL3A-Pad1) -> /FPGA/SCK_1
- U1 pad 13: unconnected-(U1A-PL10A-Pad13) -> /FPGA/SCK_2
- U1 pad 15: unconnected-(U1A-PL11A-Pad15) -> /FPGA/MOSI_2
- U1 pad 19: unconnected-(U1A-PL12A-Pad19) -> /FPGA/MISO_2
- U1 pad 2: unconnected-(U1A-PL3B-Pad2) -> /FPGA/MOSI_1
- U1 pad 26: unconnected-(U1A-PL19B-Pad26) -> /FPGA/RST
- U1 pad 28: unconnected-(U1A-PL22B-Pad28) -> /FPGA/SYNC
- U1 pad 3: unconnected-(U1A-PL4A-Pad3) -> /FPGA/MISO_1
- U1 pad 33: unconnected-(U1A-PL24B-Pad33) -> /FPGA/IRQ
- U1 pad 35: unconnected-(U1A-PL25B-Pad35) -> /FPGA/CS
- U1 pad 44: /FPGA/MCLK/CCLK -> unconnected-(U1A-PB12A-Pad44)
- U1 pad 45: /FPGA/SO/SPISO -> unconnected-(U1A-PB12B-Pad45)
- U1 pad 49: unconnected-(U1A-PB16A-Pad49) -> GND
- U1 pad 50: unconnected-(U1A-PB16B-Pad50) -> /FPGA/LED_0
- U1 pad 52: unconnected-(U1A-PB18A-Pad52) -> /FPGA/LED_1
- U1 pad 54: unconnected-(U1A-PB18B-Pad54) -> /FPGA/LED_2
- U1 pad 55: unconnected-(U1A-PB23A-Pad55) -> /FPGA/LED_3
- U1 pad 56: unconnected-(U1A-PB23B-Pad56) -> /FPGA/LED_4
- U1 pad 57: unconnected-(U1A-PB26A-Pad57) -> /FPGA/PB26A
- U1 pad 58: unconnected-(U1A-PB26B-Pad58) -> /FPGA/PB26B
- U1 pad 60: unconnected-(U1A-PB29B-Pad60) -> Net-(U1A-PB29B)
- U1 pad 63: /FPGA/IRQ -> Net-(U1A-PB31D)
- U1 pad 65: /FPGA/RST -> Net-(U1A-PB35A)
- U1 pad 67: /FPGA/SYNC -> unconnected-(U1A-PB35B-Pad67)
- U1 pad 71: /FPGA/SI/SISPI -> unconnected-(U1A-PB38B-Pad71)
- U2 pad 5: /FPGA/OSC_OUT -> GND
- U3 pad 2: /FPGA/SO/SPISO -> /FPGA/MISO_1
- U7 pad 17: /USB/RXD -> /FPGA/PB26B
- U7 pad 18: /USB/TXD -> /FPGA/PB26A
- U7 pad 6: +3.3V -> +3V3
- U7 pad 7: +3.3V -> +3V3
Routing:
- net /DONE: track 0.00 -> 38.6 mm, vias 0 -> 1
- net /INIT_N: track 0.00 -> 36.0 mm, vias 0 -> 1
- net /FPGA/CS: track 0.00 -> 28.9 mm, vias 0 -> 3
- net /PROGRAMN: track 0.00 -> 25.1 mm, vias 0 -> 1
- net /FPGA/SCK_1: track 0.00 -> 13.0 mm
- net /TDI: track 0.00 -> 12.8 mm, vias 0 -> 2
- net /TDO: track 0.00 -> 12.7 mm
- net /FPGA/IRQ: track 0.00 -> 12.7 mm, vias 0 -> 1
- net /FPGA/MOSI_1: track 0.00 -> 11.9 mm
- net /FPGA/RST: track 0.00 -> 11.6 mm
- net /FPGA/SYNC: track 0.00 -> 11.6 mm
- net /FPGA/SCK_2: track 0.00 -> 11.4 mm
- net /FPGA/MOSI_2: track 0.00 -> 11.4 mm
- net /FPGA/PB26A: track 0.00 -> 8.96 mm
- net /FPGA/PB26B: track 0.00 -> 8.14 mm
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- added copper zone on In2.Cu, net +3V3
- added copper zone on F.Cu, net GND
